Commit message: changes for python3 stuff

File: simulators/robot_files/Fetch/URDF/Fetch.urdf (robot description, URDF)
Before this commit: robot Fetch, 26 links, 25 joints
Links:
- link base_link: geometry collision mesh filename=file:///workspaces/LAMP/simulators/robot_files/Fetch/URDF/m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; visual mesh filename=file:///workspaces/LAMP/simulators/robot_files/Fetch/URDF/m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
- link bellows_link: geometry collision mesh filename=file:///workspaces/LAMP/simulators/robot_files/Fetch/URDF/m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; visual mesh filename=file:///workspaces/LAMP/simulators/robot_files/Fetch/URDF/m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
- link bellows_link2: geometry collision mesh filename=file:///workspaces/LAMP/simulators/robot_files/Fetch/URDF/m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; visual mesh filename=file:///workspaces/LAMP/simulators/robot_files/Fetch/URDF/m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
- link elbow_flex_link: geometry collision mesh filename=file:///workspaces/LAMP/simulators/robot_files/Fetch/URDF/m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; visual mesh filename=file:///workspaces/LAMP/simulators/robot_files/Fetch/URDF/m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
- link estop_link: geometry collision mesh filename=file:///workspaces/LAMP/simulators/robot_files/Fetch/URDF/m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; visual mesh filename=file:///workspaces/LAMP/simulators/robot_files/Fetch/URDF/m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
- link forearm_roll_link: geometry collision mesh filename=file:///workspaces/LAMP/simulators/robot_files/Fetch/URDF/m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; visual mesh filename=file:///workspaces/LAMP/simulators/robot_files/Fetch/URDF/m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
- link gripper_link: geometry collision mesh filename=file:///workspaces/LAMP/simulators/robot_files/Fetch/URDF/m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; visual mesh filename=file:///workspaces/LAMP/simulators/robot_files/Fetch/URDF/m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
- link head_pan_link: geometry collision mesh filename=file:///workspaces/LAMP/simulators/robot_files/Fetch/URDF/m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; visual mesh filename=file:///workspaces/LAMP/simulators/robot_files/Fetch/URDF/m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
- link head_tilt_link: geometry collision mesh filename=file:///workspaces/LAMP/simulators/robot_files/Fetch/URDF/m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; visual mesh filename=file:///workspaces/LAMP/simulators/robot_files/Fetch/URDF/m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
- link l_gripper_finger_link: geometry collision mesh filename=file:///workspaces/LAMP/simulators/robot_files/Fetch/URDF/m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; visual mesh filename=file:///workspaces/LAMP/simulators/robot_files/Fetch/URDF/m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
- link l_wheel_link: geometry collision mesh filename=file:///workspaces/LAMP/simulators/robot_files/Fetch/URDF/m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; visual mesh filename=file:///workspaces/LAMP/simulators/robot_files/Fetch/URDF/m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
- link laser_link: geometry collision mesh filename=file:///workspaces/LAMP/simulators/robot_files/Fetch/URDF/m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; visual mesh filename=file:///workspaces/LAMP/simulators/robot_files/Fetch/URDF/m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
- link r_gripper_finger_link: geometry collision mesh filename=file:///workspaces/LAMP/simulators/robot_files/Fetch/URDF/m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; visual mesh filename=file:///workspaces/LAMP/simulators/robot_files/Fetch/URDF/m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
- link r_wheel_link: geometry collision mesh filename=file:///workspaces/LAMP/simulators/robot_files/Fetch/URDF/m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; visual mesh filename=file:///workspaces/LAMP/simulators/robot_files/Fetch/URDF/m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
- link shoulder_lift_link: geometry collision mesh filename=file:///workspaces/LAMP/simulators/robot_files/Fetch/URDF/m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; visual mesh filename=file:///workspaces/LAMP/simulators/robot_files/Fetch/URDF/m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
- link shoulder_pan_link: geometry collision mesh filename=file:///workspaces/LAMP/simulators/robot_files/Fetch/URDF/m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; visual mesh filename=file:///workspaces/LAMP/simulators/robot_files/Fetch/URDF/m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
- link torso_fixed_link: geometry collision mesh filename=file:///workspaces/LAMP/simulators/robot_files/Fetch/URDF/m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; visual mesh filename=file:///workspaces/LAMP/simulators/robot_files/Fetch/URDF/m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
- link torso_lift_link: geometry collision mesh filename=file:///workspaces/LAMP/simulators/robot_files/Fetch/URDF/m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; visual mesh filename=file:///workspaces/LAMP/simulators/robot_files/Fetch/URDF/m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
- link upperarm_roll_link: geometry collision mesh filename=file:///workspaces/LAMP/simulators/robot_files/Fetch/URDF/m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; visual mesh filename=file:///workspaces/LAMP/simulators/robot_files/Fetch/URDF/m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
- link wrist_flex_link: geometry collision mesh filename=file:///workspaces/LAMP/simulators/robot_files/Fetch/URDF/m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; visual mesh filename=file:///workspaces/LAMP/simulators/robot_files/Fetch/URDF/m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
- link wrist_roll_link: geometry collision mesh filename=file:///workspaces/LAMP/simulators/robot_files/Fetch/URDF/m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; visual mesh filename=file:///workspaces/LAMP/simulators/robot_files/Fetch/URDF/m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

Commit message: fixes for visualization and init staring

File: simulators/robot_files/Fetch/URDF/Fetch.urdf (robot description, URDF)
Before this commit: robot Fetch, 26 links, 25 joints
Links:
- link base_link: geometry collision mesh filename=file://project_directory/simulators/robot_files/Fetch/URDF/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; visual mesh filename=file://project_directory/simulators/robot_files/Fetch/URDF/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
- link bellows_link: geometry collision mesh filename=file://project_directory/simulators/robot_files/Fetch/URDF/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; visual mesh filename=file://project_directory/simulators/robot_files/Fetch/URDF/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
- link bellows_link2: geometry collision mesh filename=file://project_directory/simulators/robot_files/Fetch/URDF/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; visual mesh filename=file://project_directory/simulators/robot_files/Fetch/URDF/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
- link elbow_flex_link: geometry collision mesh filename=file://project_directory/simulators/robot_files/Fetch/URDF/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; visual mesh filename=file://project_directory/simulators/robot_files/Fetch/URDF/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
- link estop_link: geometry collision mesh filename=file://project_directory/simulators/robot_files/Fetch/URDF/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; visual mesh filename=file://project_directory/simulators/robot_files/Fetch/URDF/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
- link forearm_roll_link: geometry collision mesh filename=file://project_directory/simulators/robot_files/Fetch/URDF/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; visual mesh filename=file://project_directory/simulators/robot_files/Fetch/URDF/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
- link gripper_link: geometry collision mesh filename=file://project_directory/simulators/robot_files/Fetch/URDF/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; visual mesh filename=file://project_directory/simulators/robot_files/Fetch/URDF/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
- link head_pan_link: geometry collision mesh filename=file://project_directory/simulators/robot_files/Fetch/URDF/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; visual mesh filename=file://project_directory/simulators/robot_files/Fetch/URDF/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
- link head_tilt_link: geometry collision mesh filename=file://project_directory/simulators/robot_files/Fetch/URDF/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; visual mesh filename=file://project_directory/simulators/robot_files/Fetch/URDF/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
- link l_gripper_finger_link: geometry collision mesh filename=file://project_directory/simulators/robot_files/Fetch/URDF/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; visual mesh filename=file://project_directory/simulators/robot_files/Fetch/URDF/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
- link l_wheel_link: geometry collision mesh filename=file://project_directory/simulators/robot_files/Fetch/URDF/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; visual mesh filename=file://project_directory/simulators/robot_files/Fetch/URDF/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
- link laser_link: geometry collision mesh filename=file://project_directory/simulators/robot_files/Fetch/URDF/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; visual mesh filename=file://project_directory/simulators/robot_files/Fetch/URDF/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
- link r_gripper_finger_link: geometry collision mesh filename=file://project_directory/simulators/robot_files/Fetch/URDF/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; visual mesh filename=file://project_directory/simulators/robot_files/Fetch/URDF/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
- link r_wheel_link: geometry collision mesh filename=file://project_directory/simulators/robot_files/Fetch/URDF/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; visual mesh filename=file://project_directory/simulators/robot_files/Fetch/URDF/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
- link shoulder_lift_link: geometry collision mesh filename=file://project_directory/simulators/robot_files/Fetch/URDF/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; visual mesh filename=file://project_directory/simulators/robot_files/Fetch/URDF/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
- link shoulder_pan_link: geometry collision mesh filename=file://project_directory/simulators/robot_files/Fetch/URDF/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; visual mesh filename=file://project_directory/simulators/robot_files/Fetch/URDF/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
- link torso_fixed_link: geometry collision mesh filename=file://project_directory/simulators/robot_files/Fetch/URDF/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; visual mesh filename=file://project_directory/simulators/robot_files/Fetch/URDF/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
- link torso_lift_link: geometry collision mesh filename=file://project_directory/simulators/robot_files/Fetch/URDF/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; visual mesh filename=file://project_directory/simulators/robot_files/Fetch/URDF/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
- link upperarm_roll_link: geometry collision mesh filename=file://project_directory/simulators/robot_files/Fetch/URDF/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; visual mesh filename=file://project_directory/simulators/robot_files/Fetch/URDF/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
- link wrist_flex_link: geometry collision mesh filename=file://project_directory/simulators/robot_files/Fetch/URDF/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; visual mesh filename=file://project_directory/simulators/robot_files/Fetch/URDF/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
- link wrist_roll_link: geometry collision mesh filename=file://project_directory/simulators/robot_files/Fetch/URDF/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; visual mesh filename=file://project_directory/simulators/robot_files/Fetch/URDF/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
